Commit message: Fixed Base Joint Issue

File: src/robotic_arm_urdf/urdf/robotic_arm_urdf.urdf (robot description, URDF)
Before this commit: robot robotic_arm_urdf, 7 links, 6 joints
Links:
- link Base: mass 2.03790063849228 -> 1.89486895954733
- link FIxed_plate: mass 0.182707362998648 -> 0.325739041943602
- link Gripper: mass 0.0388186179630647 -> 0.0388186179630637
- link Shoulder: mass 0.206135703604005 -> 0.206135703604
- link Wrist_rotate: mass 0.330165609400152 -> 0.330165609400149
- link Wrist_vertical: mass 0.230335497213652 -> 0.23033549720499
Joints:
- joint Base_joint: origin xyz=-0.124999999876148 -0.115000000066085 -0.0605000010000004 rpy=3.14159265358979 0 0 -> xyz=-0.000869195529410005 0.000774746946535121 0.0750000020000001 rpy=0 0 0
- joint Gripper_joint: axis 0.999621046088342 -0.0275275174552392 0 -> -0.999621046088342 0.0275275174552392 0; origin xyz=-0.0379340918072452 0.106065377730978 0.00961198872859703 rpy=3.14159265358979 0 0 -> xyz=-0.037934092087304 0.106065377723266 0.00961198872859703 rpy=3.14159265358979 0 3.14159265358979
- joint Shoulder_joint: axis 0.999621046089309 0.0275275174201498 0 -> 0.999621046089309 0.0275275174201486 0; origin xyz=0.0447330416894474 -0.0012318564762297 0.0905000009999997 rpy=3.14159265358979 0 3.14159265358979 -> xyz=0.0447197560242002 -0.00112412203816992 0.073 rpy=3.14159265358979 0 3.14159265358979
- joint Wrist_rotate_joint: axis 0.0274172576374167 -0.995617124026799 -0.0894138486379473 -> 0.0274172576374139 -0.995617124026799 -0.0894138486379424
- joint Wrist_vertical_joint: axis 0.99962 0.027528 0 -> 0.999621046088342 0.0275275174552392 0; origin xyz=-0.011442 0.41551 0.037316 rpy=0 0 0 -> xyz=-0.0114424125784452 0.415514271147883 0.0373162827874605 rpy=0 0 0
